File: cad/midipod.kicad_pcb (KiCad board)
At the start: 2 copper layers, 50.8 x 51.4 mm, 22 parts, among them IC1 ATMEGA8U2, M3 1pin, P1 ISP, P2 USB, P3 INV1, P4 SW1, Y1 Crystal

Commit message: Check electric rules passed.
Routing:
- net GND: vias 1 -> 4
Changed lines of the file:
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@@
-(kicad_pcb (version 20171130) (host pcbnew "(6.0.0-rc1-dev-1215-g431bdc7a3)")
+(kicad_pcb (version 20171130) (host pcbnew "(5.1.5-0-10_14)")
   (general
     (thickness 1.6)
     (drawings 6)
-    (tracks 118)
+    (tracks 123)
     (zones 0)
     (modules 22)
@@
   (layers
     (0 F.Cu signal)
-    (31 B.Cu signal)
-    (32 B.Adhes user hide)
-    (33 F.Adhes user hide)
-    (34 B.Paste user hide)
-    (35 F.Paste user hide)
-    (36 B.SilkS user hide)
+    (31 B.Cu signal hide)
+    (32 B.Adhes user)
+    (33 F.Adhes user)
+    (34 B.Paste user)
+    (35 F.Paste user)
+    (36 B.SilkS user)
     (37 F.SilkS user)
-    (38 B.Mask user hide)
-    (39 F.Mask user hide)
+    (38 B.Mask user)
+    (39 F.Mask user)
     (40 Dwgs.User user)
     (41 Cmts.User user)
@@
     (mod_text_size 1 1)
     (mod_text_width 0.15)
-    (pad_size 1.6 0.52)
-    (pad_drill 0)
+    (pad_size 4.064 4.064)
+    (pad_drill 3.048)
     (pad_to_mask_clearance 0)
     (solder_mask_min_width 0.25)
     (aux_axis_origin 129.286 124.079)
     (grid_origin 129.286 124.079)
-    (visible_elements FFFFF77F)
+    (visible_elements FEFDB63F)
     (pcbplotparams
       (layerselection 0x000f0_80000001)
@@
   (segment (start 164.973 106.299) (end 164.973 116.586) (width 0.25) (layer B.Cu) (net 1))
   (segment (start 161.163 102.489) (end 164.973 106.299) (width 0.25) (layer B.Cu) (net 1))
-  (segment (start 152.976 109.709) (end 150.514 109.709) (width 0.25) (layer F.Cu) (net 1) (status 10))
   (segment (start 159.766 102.489) (end 155.702 102.489) (width 0.25) (layer B.Cu) (net 1))
   (segment (start 155.702 102.489) (end 154.432 103.759) (width 0.25) (layer B.Cu) (net 1))
@@
   (segment (start 163.576 89.209) (end 163.576 89.059) (width 0.25) (layer F.Cu) (net 1) (status 30))
   (segment (start 163.576 89.059) (end 166.656 89.059) (width 0.25) (layer F.Cu) (net 1) (status 10))
-  (segment (start 144.145 103.34) (end 150.514 109.709) (width 0.25) (layer F.Cu) (net 1))
-  (segment (start 144.145 98.933) (end 144.145 103.34) (width 0.25) (layer F.Cu) (net 1))
   (segment (start 153.314752 81.62798) (end 153.314752 81.635248) (width 0.25) (layer F.Cu) (net 1) (status 30))
   (segment (start 153.314752 81.635248) (end 151.003 83.947) (width 0.25) (layer F.Cu) (net 1) (status 10))
-  (segment (start 151.003 83.947) (end 147.955 83.947) (width 0.25) (layer F.Cu) (net 1))
-  (segment (start 147.955 83.947) (end 146.431 85.471) (width 0.25) (layer F.Cu) (net 1))
-  (segment (start 146.431 85.471) (end 146.431 96.647) (width 0.25) (layer F.Cu) (net 1))
-  (segment (start 146.431 96.647) (end 144.145 98.933) (width 0.25) (layer F.Cu) (net 1))
-  (via (at 157.626 108.60664) (size 0.6) (drill 0.4) (layers F.Cu B.Cu) (net 2))
+  (segment (start 151.003 83.947) (end 148.082 83.947) (width 0.25) (layer F.Cu) (net 1))
+  (segment (start 148.082 83.947) (end 147.955 83.947) (width 0.25) (layer F.Cu) (net 1))
+  (segment (start 144.145 103.34) (end 150.514 109.709) (width 0.25) (layer F.Cu) (net 1))
+  (segment (start 144.145 98.552) (end 144.145 103.34) (width 0.25) (layer F.Cu) (net 1))
+  (segment (start 146.05 96.647) (end 144.145 98.552) (width 0.25) (layer F.Cu) (net 1))
+  (segment (start 146.05 85.471) (end 146.05 96.647) (width 0.25) (layer F.Cu) (net 1))
+  (segment (start 147.574 83.947) (end 146.05 85.471) (width 0.25) (layer F.Cu) (net 1))
+  (segment (start 150.514 109.709) (end 152.976 109.709) (width 0.25) (layer F.Cu) (net 1))
+  (segment (start 148.082 83.947) (end 147.574 83.947) (width 0.25) (layer F.Cu) (net 1))
   (segment (start 157.626 105.859) (end 157.626 108.60664) (width 0.25) (layer F.Cu) (net 2) (status 10))
   (segment (start 152.976 108.909) (end 151.3902 108.909) (width 0.25) (layer F.Cu) (net 2) (status 10))
+  (via (at 155.956 110.109) (size 0.6) (drill 0.4) (layers F.Cu B.Cu) (net 2))
+  (via (at 157.226 108.839) (size 0.6) (drill 0.4) (layers F.Cu B.Cu) (net 2))
+  (via (at 157.226 111.379) (size 0.6) (drill 0.4) (layers F.Cu B.Cu) (net 2))
+  (via (at 158.496 110.109) (size 0.6) (drill 0.4) (layers F.Cu B.Cu) (net 2))
   (segment (start 152.976 107.309) (end 152.406 107.309) (width 0.25) (layer F.Cu) (net 3) (status 30))
   (segment (start 152.406 107.309) (end 150.876 105.779) (width 0.25) (layer F.Cu) (net 3) (status 10))
